File: pcb/qwertyxpansion.kicad_sch (KiCad schematic)
At the start: 72 parts, among them SW1 Q, SW10 P, SW11 A, SW12 S, SW13 D, SW14 F, SW15 G, SW16 H, SW17 J, SW18 K, SW19 L, SW2 W, SW20 Z, SW21 X, SW22 C, SW23 V, SW24 B, SW25 N, SW26 M, SW27 ,, SW28 ., SW29 SW_Push_45deg, SW3 E, SW30 SW_Push_45deg, SW31 SW_Push_45deg, SW32 SW_Push_45deg, SW33 SW_Push_45deg, SW4 R, SW5 T, SW6 Y, SW7 U, SW8 I, SW9 O

Commit message: stuffs
Parts:
- D1, D10, D11, D12, D13, D14, D15, D16, D17, D18, D19, D2, D20, D21, D22, D23, D24, D25, D26, D27, D28, D29, D3, D30, D31, D32, D33, D4, D5, D6, D7, D8, D9: LCSC Part # (none) -> C28646371
- D34: LCSC Part # (none) -> C20608782
- R1: LCSC Part # (none) -> C2909383
- R2: LCSC Part # (none) -> C140197
- R3: LCSC Part # (none) -> C25102
- SW1: value Q -> SW_Push_45deg
- SW10: value P -> SW_Push_45deg
- SW11: value A -> SW_Push_45deg
- SW12: value S -> SW_Push_45deg
- SW13: value D -> SW_Push_45deg
- SW14: value F -> SW_Push_45deg
- SW15: value G -> SW_Push_45deg
- SW16: value H -> SW_Push_45deg
- SW17: value J -> SW_Push_45deg
- SW18: value K -> SW_Push_45deg
- SW19: value L -> SW_Push_45deg
- SW2: value W -> SW_Push_45deg
- SW20: value Z -> SW_Push_45deg
- SW21: value X -> SW_Push_45deg
- SW22: value C -> SW_Push_45deg
- SW23: value V -> SW_Push_45deg
- SW24: value B -> SW_Push_45deg
- SW25: value N -> SW_Push_45deg
- SW26: value M -> SW_Push_45deg
- SW27: value , -> SW_Push_45deg
- SW28: value . -> SW_Push_45deg
- SW3: value E -> SW_Push_45deg
- SW4: value R -> SW_Push_45deg
- SW5: value T -> SW_Push_45deg
- SW6: value Y -> SW_Push_45deg
- SW7: value U -> SW_Push_45deg
- SW8: value I -> SW_Push_45deg
- SW9: value O -> SW_Push_45deg
