File: pcb/qwertyxpansion.kicad_pcb (KiCad board)
At the start: 2 copper layers, 52 x 32 mm, 75 parts, among them SW1 Q, SW10 P, SW11 A, SW12 S, SW13 D, SW14 F, SW15 G, SW16 H, SW17 J, SW18 K, SW19 L, SW2 W, SW20 Z, SW21 X, SW22 C, SW23 V, SW24 B, SW25 N, SW26 M, SW27 ,, SW28 ., SW29 SW_Push_45deg, SW3 E, SW30 SW_Push_45deg, SW31 SW_Push_45deg, SW32 SW_Push_45deg, SW33 SW_Push_45deg, SW4 R, SW5 T, SW6 Y, SW7 U, SW8 I, SW9 O

Commit message: files and driver
Parts:
- added G***: LOGO, LOGO, B.Cu at (180.9, 119.1)
Other:
- board text added: "GitHub"
- board text added: "qwerty"
- board text removed: "Keeb"
